Commit message: Update the joint of the camera

File: gara_project/urdf/gara_description.xacro (robot description, xacro)
@@ -4,4 +4,5 @@
 	<link name='camera_link'></link>
  	<joint name="base_link_joint" type="fixed">
+		<origin xyz="0 0 1.0" rpy="0 0 0" />
     		<parent link="base_link"/>
 		<child link="camera_link"/>

Commit message: Added realsense configuration file and other minor changes

File: gara_project/urdf/gara_description.xacro (robot description, xacro)
@@ -4,5 +4,5 @@
 	<link name='camera_link'></link>
  	<joint name="base_link_joint" type="fixed">
-		<origin xyz="0 0 1.0" rpy="0 0 0" />
+		<origin xyz="0.28 0 0.8" rpy="0 0 0" />
     		<parent link="base_link"/>
 		<child link="camera_link"/>

Commit message: Configure the IMU calibration

File: gara_project/urdf/gara_description.xacro (robot description, xacro)
@@ -3,8 +3,15 @@
 	<link name='base_link'></link>
 	<link name='camera_link'></link>
+	<link name="imu_link"></link>
  	<joint name="base_link_joint" type="fixed">
-		<origin xyz="0.28 0 0.8" rpy="0 0 0" />
+		<origin xyz="0 0 0" rpy="0 0 0" />
     		<parent link="base_link"/>
 		<child link="camera_link"/>
 	</joint>
+ 	<!-- IMU Joint 	-->
+	<joint name="imu_joint" type="fixed">
+		<origin xyz="0 0 0" rpy="0 0 0"/>
+		<parent link="base_link"/>
+		<child link="imu_link"/>
+  </joint>
 </robot>

Commit message: Localization setup

File: gara_project/urdf/gara_description.xacro (robot description, xacro)
@@ -2,16 +2,9 @@
 <robot name="gara" xmlns:xacro="http://www.ros.org/wiki/xacro">
 	<link name='base_link'></link>
-	<link name='camera_link'></link>
 	<link name="imu_link"></link>
- 	<joint name="base_link_joint" type="fixed">
-		<origin xyz="0 0 0" rpy="0 0 0" />
-    		<parent link="base_link"/>
-		<child link="camera_link"/>
-	</joint>
- 	<!-- IMU Joint 	-->
 	<joint name="imu_joint" type="fixed">
 		<origin xyz="0 0 0" rpy="0 0 0"/>
 		<parent link="base_link"/>
 		<child link="imu_link"/>
-  </joint>
+  	</joint>
 </robot>
