Commit message: Including Robot localization in simulation

File: gara_simulation/urdf/gara.xacro (robot description, xacro)
@@ -1,87 +1,65 @@
 <?xml version="1.0"?>
+<!-- TODO CHECK INERTIAL COLLISION AND FIXED JOINTS" -->
 <robot name="gara" xmlns:xacro="http://ros.org/wiki/xacro">
 	<xacro:include filename="$(find gara_simulation)/urdf/gara.gazebo" />
-	<gazebo reference="chassis">
-  		<material>Gazebo/Black</material>
-	</gazebo>
 	<!-- Base Link -->
-  	<link name="base_link"></link>
+  <link name="base_link"></link>
+	<!--Robot chassis Link-->
+	<link name="chassis">
+  	<visual>
+			<geometry>
+		  	<cylinder length="0.018" radius="0.257"/>
+			</geometry>
+  	</visual>
+		<collision>
+  			<geometry>
+    			<cylinder length="0.018" radius="0.257"/>
+  			</geometry>
+		</collision>
+		<inertial>
+  			<mass value="20"/>
+  			<inertia 	ixx="0.330785" ixy="0.0" ixz="0.0"
+								 	iyy="0.330785" iyz="0.0"
+									izz="0.66049"/>
+		</inertial>
+	</link>
 	<!--Robot chassis Joint-->
-  	<joint name="base_link_joint" type="fixed">
-    		<origin xyz="0 0 0" rpy="0 0 0" />
-    		<parent link="base_link"/>
-    		<child link="chassis" />
-  	</joint>
-	<!--Robot chassis Link-->
-  	<link name="chassis">
-    		<visual>
-			<!--  TODO
-      			<geometry>
-        			<mesh filename="package://gara_simulation/meshes/gara.dae"/>
-      			</geometry>
-			-->
-			<origin rpy="0 0 0" xyz="0 0 0.0"/>
-			<geometry>
-        			<cylinder length="0.018" radius="0.257"/>
-      			</geometry>
-    		</visual>
-    		<collision>
-      			<origin rpy="0 0 0" xyz="0 0 0.0"/>
-      			<geometry>
-        			<cylinder length="0.018" radius="0.257"/>
-      			</geometry>
-    		</collision>
-    		<inertial>
-      			<mass value="20"/>
-      			<origin xyz="0 0 0"/>
-      			<inertia ixx="0.330785" ixy="0.0" ixz="0.0" iyy="0.330785" iyz="0.0" izz="0.66049"/>
-    		</inertial>
-  	</link>
-  	<!--Caster Joint-->
-  	<joint name="center_wheel_joint" type="fixed">
-    		<parent link="chassis"/>
-    		<child link="center_wheel"/>
-		<axis xyz="0 0 0" rpy="0 0 0">
-		</axis>
+  <joint name="base_link_joint" type="fixed">
+		<origin xyz="0 0 0.125" rpy="0 0 0" />
+    <parent link="base_link"/>
+    <child link="chassis" />
+  </joint>
+	<!--Caster Link-->
+	<link name="center_wheel">
+		<visual>
+				<geometry>
+					<sphere radius="0.058"/>
+				</geometry>
+		</visual>
+		<collision>
+ 			<geometry>
+    			<sphere radius="0.058"/>
+ 			</geometry>
+		</collision>
+		<inertial>
+ 			<mass value="1"/>
+ 			<inertia 	ixx="0.001346" ixy="0.0" ixz="0.0"
+								iyy="0.001346" iyz="0.0"
+								izz="0.001346"/>
+		</inertial>
+	</link>
+	<!--Caster Joint-->
+	<joint name="center_wheel_joint" type="fixed">
 		<origin xyz="0.14 0.0 -0.067" rpy="0 0 0"/>
-		<limit effort="10000" velocity="1000"/>
-  	</joint>
-  	<!--Caster Link-->
-  	<link name="center_wheel">
-    		<visual>
-      			<origin xyz="0.0 0 0" rpy="0 0 0"/>
-      			<geometry>
-        			<sphere radius="0.058"/>
-      			</geometry>
-      			<material name="black"/>
-    		</visual>
-    		<collision>
-      			<origin xyz="0.0 0 0" rpy="0 0 0"/>
-     			<geometry>
-        			<sphere radius="0.058"/>
-     			</geometry>
-    		</collision>
-    		<inertial>
-     			<mass value="1"/>
-     			<inertia ixx="0.004" ixy="0.0" ixz="0.0" iyy="0.004" iyz="0.0" izz="0.004"/>
-    		</inertial>
-  	</link>
-	<!-- Left Wheel Joint  -->
-	<joint name="left_wheel_hinge" type="continuous" >
-		<parent link="chassis"/>
-		<child link="left_wheel"/>
-		<axis xyz="0 1 0" rpy="0 0 0">
-		</axis>
-		<origin xyz="-0.182 0.285 0" rpy="0 0 0"/>
-		<limit effort="10000" velocity="1000"/>
+		<parent link="chassis"/>
+		<child link="center_wheel"/>
 	</joint>
 	<!-- Left Wheel Link  -->
 	<link name='left_wheel'>
-		<visual name='left_wheel_visual'>
-			<origin xyz="0.0 0 0" rpy="0 1.5707 1.5707"/>
-			<geometry>
-				<cylinder radius="0.125" length="0.05"/>
-			</geometry>
-			<material name="yellow"/>
+		<visual>
+			<origin xyz="0.0 0 0" rpy="0 1.5707 1.5707"/>
+			<geometry>
+				<cylinder radius="0.125" length="0.05"/>
+			</geometry>
 		</visual>
 		<collision name='collision'>
@@ -92,6 +70,6 @@
 		</collision>
 		<inertial>
+			<origin xyz="0.0 0 0" rpy="0 1.5707 1.5707"/>
 			<mass value="2"/>
-			<origin xyz="0.0 0 0" rpy="0 1.5707 1.5707"/>
 			<inertia
 			  ixx="0.008229" ixy="0" ixz="0"
@@ -101,21 +79,18 @@
 		</inertial>
 	</link>
-	<!-- Right Wheel Joint -->
-	<joint name="right_wheel_hinge" type="continuous" >
-		<parent link="chassis"/>
-		<child link="right_wheel"/>
-		<axis xyz="0 1 0" rpy="0 0 0">
-		</axis>
-		<origin xyz="-0.182 -0.285 0" rpy="0 0 0"/>
-		<limit effort="10000" velocity="1000"/>
+	<!-- Left Wheel Joint  -->
+	<joint name="left_wheel_hinge" type="continuous">
+		<axis xyz="0 1 0" rpy="0 0 0"/>
+		<origin xyz="-0.182 0.285 0" rpy="0 0 0"/>
+		<parent link="chassis"/>
+		<child link="left_wheel"/>
 	</joint>
 	<!-- Right Wheel Link -->
 	<link name='right_wheel'>
-		<visual name='right_wheel_visual'>
-			<origin xyz="0.0 0 0" rpy="0 1.5707 1.5707"/>
-			<geometry>
-				<cylinder radius="0.125" length="0.05"/>
-			</geometry>
-			<material name="yellow"/>
+		<visual >
+			<origin xyz="0.0 0 0" rpy="0 1.5707 1.5707"/>
+			<geometry>
+				<cylinder radius="0.125" length="0.05"/>
+			</geometry>
 		</visual>
 		<collision name='collision'>
@@ -126,6 +101,6 @@
 		</collision>
 		<inertial>
+			<origin xyz="0.0 0 0" rpy="0 1.5707 1.5707"/>
 			<mass value="2"/>
-			<origin xyz="0.0 0 0" rpy="0 1.5707 1.5707"/>
 			<inertia
 			  ixx="0.008229" ixy="0" ixz="0"
@@ -135,22 +110,21 @@
 		</inertial>
 	</link>
-	<!-- Mast Joint -->
-	<joint name="mast_hinge" type="fixed" >
-		<parent link="chassis"/>
-		<child link="mast"/>
-		<axis xyz="0 0 0" rpy="0 0 0"/>
-		<origin xyz="0 0 0.559" rpy="0 0 0"/>
+	<!-- Right Wheel Joint -->
+	<joint name="right_wheel_hinge" type="continuous" >
+		<axis xyz="0 1 0" rpy="0 0 0"/>
+		<origin xyz="-0.182 -0.285 0" rpy="0 0 0"/>
+		<parent link="chassis"/>
+		<child link="right_wheel"/>
 	</joint>
 	<!-- Mast Link -->
 	<link name='mast'>
 		<visual name='mast_visual'>
-			<origin xyz="0.0 0 0" rpy="0 0 0"/>
+			<origin xyz="0.0 0 -0.559" rpy="0 0 0"/>
 			<geometry>
 				<cylinder radius="0.02" length="1.1"/>
 			</geometry>
-			<material name="yellow"/>
 		</visual>
 		<collision name='collision'>
-			<origin xyz="0.0 0 0" rpy="0 0 0"/>
+			<origin xyz="0.0 0 -0.559" rpy="0 0 0"/>
 			<geometry>
 				<cylinder radius="0.02" length="1.1"/>
@@ -159,5 +133,4 @@
 		<inertial>
 			<mass value="2"/>
-			<origin xyz="0.0 0 0" rpy="0 0 0"/>
 			<inertia
 			  ixx="0.201867" ixy="0" ixz="0"
@@ -167,65 +140,96 @@
 		</inertial>
 	</link>
+	<!-- Mast Joint -->
+	<joint name="mast_hinge" type="fixed" >
+		<origin xyz="0 0 1.1" rpy="0 0 0"/>
+		<parent link="chassis"/>
+		<child link="mast"/>
+	</joint>
+	<!-- Camera Link -->
+	<link name="camera_link">
+		<visual>
+  			<geometry>
+					<box size="0.025 0.085 0.01"/>
+  			</geometry>
+		</visual>
+		<collision>
+  			<origin xyz="0 0 0" rpy="0 0 0"/>
+  			<geometry>
+				<box size="0.025 0.085 0.01"/>
+  			</geometry>
+		</collision>
+		<inertial>
+  			<mass value="1e-5" />
+  			<inertia 	ixx="1e-6" ixy="0" ixz="0"
+									iyy="1e-6" iyz="0"
+									izz="1e-6" />
+		</inertial>
+	</link>
 	<!-- Camera Joint -->
-  	<joint name="camera_joint" type="fixed">
-    		<axis xyz="0 1 0" />
-    		<origin xyz="0.09 0 0.85" rpy="0 0 0"/>
-    		<parent link="chassis"/>
-    		<child link="camera_link"/>
-  	</joint>
-  	<!-- Camera Link -->
-  	<link name="camera_link">
-    		<visual>
-      			<origin xyz="0 0 0" rpy="0 0 0"/>
-      			<geometry>
-    				<box size="0.025 0.085 0.01"/>
-      			</geometry>
-    		</visual>
-    		<collision>
-      			<origin xyz="0 0 0" rpy="0 0 0"/>
-      			<geometry>
-    				<box size="0.025 0.085 0.01"/>
-      			</geometry>
-    		</collision>
-    		<inertial>
-      			<mass value="1e-5" />
-      			<origin xyz="0 0 0" rpy="0 0 0"/>
-      			<inertia ixx="1e-6" ixy="0" ixz="0" iyy="1e-6" iyz="0" izz="1e-6" />
-    		</inertial>
-  	</link>
+	<joint name="camera_joint" type="fixed">
+		<origin xyz="0.09 0 0.85" rpy="0 0 0"/>
+		<parent link="chassis"/>
+		<child link="camera_link"/>
+	</joint>
+	<!-- Camera RGBD Link -->
+	<link name='camera_rgbd_frame'></link>
 	<!-- Camera RGBD Joint -->
 	<joint name="camera_rgbd_joint" type="fixed" >
-    		<parent link="camera_link"/>
-    		<child link="camera_rgbd_frame"/>
-    		<origin xyz="0 0 0" rpy="-1.5707963267948966 0 -1.5707963267948966"/>
-  	</joint>
-	<!-- Camera RGBD Link -->
-	<link name='camera_rgbd_frame'></link>
+		<origin xyz="0 0 0" rpy="-1.5707963267948966 0 -1.5707963267948966"/>
+  	<parent link="camera_link"/>
+    <child link="camera_rgbd_frame"/>
+  </joint>
+	<!-- Hokuyo Laser Link -->
+	<link name="hokuyo_link">
+  		<visual>
+    			<origin xyz="0 0 0" rpy="0 0 0"/>
+    			<geometry>
+      			<mesh filename="package://gara_simulation/meshes/hokuyo.dae"/>
+    			</geometry>
+  		</visual>
+  		<collision>
+    			<geometry>
+      			<box size="0.1 0.1 0.1"/>
+    			</geometry>
+  		</collision>
+  		<inertial>
+    			<mass value="1e-5" />
+    			<inertia 	ixx="1e-6" ixy="0" ixz="0"
+										iyy="1e-6" iyz="0"
+										izz="1e-6" />
+  		</inertial>
+	</link>
  	<!-- Hokuyo Laser Joint -->
 	<joint name="hokuyo_joint" type="fixed">
-    		<axis xyz="0 1 0" />
-    		<origin xyz="0 0 1.1" rpy="0 0 0"/>
-    		<parent link="chassis"/>
-    		<child link="hokuyo_link"/>
-  	</joint>
-  	<!-- Hokuyo Laser Link -->
-  	<link name="hokuyo_link">
-    		<visual>
-      			<origin xyz="0 0 0" rpy="0 0 0"/>
-      			<geometry>
-        			<mesh filename="package://gara_simulation/meshes/hokuyo.dae"/>
-      			</geometry>
-    		</visual>
-    		<collision>
-      			<origin xyz="0 0 0" rpy="0 0 0"/>
-      			<geometry>
-        			<box size="0.1 0.1 0.1"/>
-      			</geometry>
-    		</collision>
-    		<inertial>
-      			<mass value="1e-5" />
-      			<origin xyz="0 0 0" rpy="0 0 0"/>
-      			<inertia ixx="1e-6" ixy="0" ixz="0" iyy="1e-6" iyz="0" izz="1e-6" />
-    		</inertial>
-  	</link>
+    	<axis xyz="0 1 0" />
+  		<origin xyz="0 0 1.1" rpy="0 0 0"/>
+  		<parent link="chassis"/>
+  		<child link="hokuyo_link"/>
+  </joint>
+	<!-- Hokuyo Laser Link -->
+	<link name="imu_link">
+		<visual>
+				<geometry>
+					<box size="0.01 0.01 0.01"/>
+				</geometry>
+		</visual>
+		<collision>
+  			<geometry>
+    			<box size="0.01 0.01 0.01"/>
+  			</geometry>
+		</collision>
+		<inertial>
+  			<mass value="1e-5" />
+  			<inertia 	ixx="1e-6" ixy="0" ixz="0"
+									iyy="1e-6" iyz="0"
+									izz="1e-6" />
+		</inertial>
+	</link>
+ 	<!-- IMU Joint -->
+	<joint name="imu_joint" type="fixed">
+		<axis xyz="0 1 0" />
+		<origin xyz="-0.2 0 0" rpy="0 0 0"/>
+		<parent link="chassis"/>
+		<child link="imu_link"/>
+  </joint>
 </robot>

Commit message: ROS controller configured

File: gara_simulation/urdf/gara.xacro (robot description, xacro)
@@ -2,63 +2,70 @@
 <!-- TODO CHECK INERTIAL COLLISION AND FIXED JOINTS" -->
 <robot name="gara" xmlns:xacro="http://ros.org/wiki/xacro">
+	<xacro:include filename="$(find gara_simulation)/urdf/macros.xacro" />
 	<xacro:include filename="$(find gara_simulation)/urdf/gara.gazebo" />
+	<xacro:include filename="$(find gara_simulation)/urdf/gara_dimensions.xacro" />
 	<!-- Base Link -->
-  <link name="base_link"></link>
-	<!--Robot chassis Link-->
+	<link name="base_link"></link>
+	<!--Robot chassis Link 	-->
 	<link name="chassis">
-  	<visual>
-			<geometry>
-		  	<cylinder length="0.018" radius="0.257"/>
-			</geometry>
-  	</visual>
-		<collision>
-  			<geometry>
-    			<cylinder length="0.018" radius="0.257"/>
-  			</geometry>
-		</collision>
-		<inertial>
-  			<mass value="20"/>
-  			<inertia 	ixx="0.330785" ixy="0.0" ixz="0.0"
-								 	iyy="0.330785" iyz="0.0"
-									izz="0.66049"/>
-		</inertial>
-	</link>
-	<!--Robot chassis Joint-->
-  <joint name="base_link_joint" type="fixed">
-		<origin xyz="0 0 0.125" rpy="0 0 0" />
-    <parent link="base_link"/>
-    <child link="chassis" />
-  </joint>
-	<!--Caster Link-->
+  		<visual>
+			<origin xyz="0 0 ${wheelRadius}" rpy="0 0 0" />
+			<geometry>
+		  	<cylinder length="${chassisWidth}" radius="${chassisRadius}"/>
+			</geometry>
+  		</visual>
+		<collision>
+			<origin xyz="0 0 ${wheelRadius}" rpy="0 0 0" />
+  			<geometry>
+    			<cylinder length="${chassisWidth}" radius="${chassisRadius}"/>
+  			</geometry>
+		</collision>
+		<inertial>
+			<origin xyz="0 0 ${wheelRadius}" rpy="0 0 0" />
+  			<mass value="${chassisMass}"/>
+			<cylinder_inertia
+				m="${chassisMass}"
+				r="${chassisRadius}"
+				h="${chassisWidth}"/>
+		</inertial>
+	</link>
+	<!--Robot chassis Joint -->
+  	<joint name="base_link_joint" type="fixed">
+		<origin xyz="0 0 0" rpy="0 0 0" />
+    	<parent link="base_link"/>
+    	<child link="chassis" />
+  	</joint>
+	<!--Caster Link -->
 	<link name="center_wheel">
 		<visual>
+				<origin xyz="0 0 0" rpy="0 0 0"/>
 				<geometry>
-					<sphere radius="0.058"/>
+					<sphere radius="${casterRadius}"/>
 				</geometry>
 		</visual>
 		<collision>
  			<geometry>
-    			<sphere radius="0.058"/>
+    			<sphere radius="${casterRadius}"/>
  			</geometry>
 		</collision>
 		<inertial>
- 			<mass value="1"/>
- 			<inertia 	ixx="0.001346" ixy="0.0" ixz="0.0"
-								iyy="0.001346" iyz="0.0"
-								izz="0.001346"/>
-		</inertial>
-	</link>
-	<!--Caster Joint-->
+ 			<mass value="${casterMass}"/>
+			<sphere_inertia
+				m="${casterMass}"
+				r="${casterRadius}"/>
+		</inertial>
+	</link>
+	<!--Caster Joint -->
 	<joint name="center_wheel_joint" type="fixed">
-		<origin xyz="0.14 0.0 -0.067" rpy="0 0 0"/>
+		<origin xyz="0.14 0 ${casterRadius}" rpy="0 0 0"/>
 		<parent link="chassis"/>
 		<child link="center_wheel"/>
 	</joint>
-	<!-- Left Wheel Link  -->
+	<!-- Left Wheel Link  	-->
 	<link name='left_wheel'>
 		<visual>
 			<origin xyz="0.0 0 0" rpy="0 1.5707 1.5707"/>
 			<geometry>
-				<cylinder radius="0.125" length="0.05"/>
+				<cylinder radius="${wheelRadius}" length="${wheelWidth}"/>
 			</geometry>
 		</visual>
@@ -66,23 +73,23 @@
 			<origin xyz="0.0 0 0" rpy="0 1.5707 1.5707"/>
 			<geometry>
-				<cylinder radius="0.125" length="0.05"/>
-			</geometry>
-		</collision>
-		<inertial>
-			<origin xyz="0.0 0 0" rpy="0 1.5707 1.5707"/>
-			<mass value="2"/>
-			<inertia
-			  ixx="0.008229" ixy="0" ixz="0"
-			  iyy="0.008229" iyz="0"
-			  izz="0.015625"
-			/>
-		</inertial>
-	</link>
-	<!-- Left Wheel Joint  -->
+				<cylinder radius="${wheelRadius}" length="${wheelWidth}"/>
+			</geometry>
+		</collision>
+		<inertial>
+			<origin xyz="0.0 0 0" rpy="0 1.5707 1.5707"/>
+			<mass value="${wheelMass}"/>
+			<cylinder_inertia
+				m="${wheelMass}"
+				r="${wheelRadius}"
+				h="${wheelWidth}"/>
+		</inertial>
+	</link>
+	<!-- Left Wheel Joint -->
 	<joint name="left_wheel_hinge" type="continuous">
 		<axis xyz="0 1 0" rpy="0 0 0"/>
-		<origin xyz="-0.182 0.285 0" rpy="0 0 0"/>
+		<origin xyz="-0.182 0.285 ${wheelRadius}" rpy="0 0 0"/>
 		<parent link="chassis"/>
 		<child link="left_wheel"/>
+		<limit effort="10000.0" velocity="10000.0"/>
 	</joint>
 	<!-- Right Wheel Link -->
@@ -91,5 +98,5 @@
 			<origin xyz="0.0 0 0" rpy="0 1.5707 1.5707"/>
 			<geometry>
-				<cylinder radius="0.125" length="0.05"/>
+				<cylinder radius="${wheelRadius}" length="${wheelWidth}"/>
 			</geometry>
 		</visual>
@@ -97,15 +104,14 @@
 			<origin xyz="0.0 0 0" rpy="0 1.5707 1.5707"/>
 			<geometry>
-				<cylinder radius="0.125" length="0.05"/>
-			</geometry>
-		</collision>
-		<inertial>
-			<origin xyz="0.0 0 0" rpy="0 1.5707 1.5707"/>
-			<mass value="2"/>
-			<inertia
-			  ixx="0.008229" ixy="0" ixz="0"
-			  iyy="0.008229" iyz="0"
-			  izz="0.015625"
-			/>
+				<cylinder radius="${wheelRadius}" length="${wheelWidth}"/>
+			</geometry>
+		</collision>
+		<inertial>
+			<origin xyz="0.0 0 0" rpy="0 1.5707 1.5707"/>
+			<mass value="${wheelMass}"/>
+			<cylinder_inertia
+				m="${wheelMass}"
+				r="${wheelRadius}"
+				h="${wheelWidth}"/>
 		</inertial>
 	</link>
@@ -113,7 +119,8 @@
 	<joint name="right_wheel_hinge" type="continuous" >
 		<axis xyz="0 1 0" rpy="0 0 0"/>
-		<origin xyz="-0.182 -0.285 0" rpy="0 0 0"/>
+		<origin xyz="-0.182 -0.285 ${wheelRadius}" rpy="0 0 0"/>
 		<parent link="chassis"/>
 		<child link="right_wheel"/>
+		<limit effort="10000.0" velocity="10000.0"/>
 	</joint>
 	<!-- Mast Link -->
@@ -132,15 +139,15 @@
 		</collision>
 		<inertial>
+			<origin xyz="0 0 1.1" rpy="0 0 0"/>
 			<mass value="2"/>
-			<inertia
-			  ixx="0.201867" ixy="0" ixz="0"
-			  iyy="0.201867" iyz="0"
-			  izz="0.0004"
-			/>
+			<cylinder_inertia
+				m="0.1"
+				r="0.02"
+				h="1.1"/>
 		</inertial>
 	</link>
 	<!-- Mast Joint -->
 	<joint name="mast_hinge" type="fixed" >
-		<origin xyz="0 0 1.1" rpy="0 0 0"/>
+		<origin xyz="0 0 ${wheelRadius+1.1}" rpy="0 0 0"/>
 		<parent link="chassis"/>
 		<child link="mast"/>
@@ -160,8 +167,10 @@
 		</collision>
 		<inertial>
-  			<mass value="1e-5" />
-  			<inertia 	ixx="1e-6" ixy="0" ixz="0"
-									iyy="1e-6" iyz="0"
-									izz="1e-6" />
+			<mass value="0.1" />
+			<box_inertia
+				m="0.1"
+				x="0.025"
+				y="0.085"
+				z="0.01"/>
 		</inertial>
 	</link>
@@ -172,13 +181,13 @@
 		<child link="camera_link"/>
 	</joint>
-	<!-- Camera RGBD Link -->
+	<!-- Camera RGBD Link 	-->
 	<link name='camera_rgbd_frame'></link>
 	<!-- Camera RGBD Joint -->
 	<joint name="camera_rgbd_joint" type="fixed" >
 		<origin xyz="0 0 0" rpy="-1.5707963267948966 0 -1.5707963267948966"/>
-  	<parent link="camera_link"/>
-    <child link="camera_rgbd_frame"/>
-  </joint>
-	<!-- Hokuyo Laser Link -->
+  		<parent link="camera_link"/>
+    	<child link="camera_rgbd_frame"/>
+  	</joint>
+	<!-- Hokuyo Laser Link 	-->
 	<link name="hokuyo_link">
   		<visual>
@@ -194,8 +203,10 @@
   		</collision>
   		<inertial>
-    			<mass value="1e-5" />
-    			<inertia 	ixx="1e-6" ixy="0" ixz="0"
-										iyy="1e-6" iyz="0"
-										izz="1e-6" />
+		  	<mass value="0.1" />
+			<box_inertia
+				m="0.1"
+				x="0.1"
+				y="0.1"
+				z="0.1"/>
   		</inertial>
 	</link>
@@ -206,11 +217,11 @@
   		<parent link="chassis"/>
   		<child link="hokuyo_link"/>
-  </joint>
+  	</joint>
 	<!-- Hokuyo Laser Link -->
 	<link name="imu_link">
 		<visual>
-				<geometry>
-					<box size="0.01 0.01 0.01"/>
-				</geometry>
+			<geometry>
+				<box size="0.01 0.01 0.01"/>
+			</geometry>
 		</visual>
 		<collision>
@@ -220,16 +231,18 @@
 		</collision>
 		<inertial>
-  			<mass value="1e-5" />
-  			<inertia 	ixx="1e-6" ixy="0" ixz="0"
-									iyy="1e-6" iyz="0"
-									izz="1e-6" />
-		</inertial>
-	</link>
- 	<!-- IMU Joint -->
+		  	<mass value="0.1" />
+			<box_inertia
+				m="0.1"
+				x="0.01"
+				y="0.01"
+				z="0.01"/>
+		</inertial>
+	</link>
+ 	<!-- IMU Joint 	-->
 	<joint name="imu_joint" type="fixed">
 		<axis xyz="0 1 0" />
-		<origin xyz="-0.2 0 0" rpy="0 0 0"/>
+		<origin xyz="-0.2 0 ${wheelRadius}" rpy="0 0 0"/>
 		<parent link="chassis"/>
 		<child link="imu_link"/>
-  </joint>
+  	</joint>
 </robot>

Commit message: Localization clean up and confituration rtabmap

File: gara_simulation/urdf/gara.xacro (robot description, xacro)
@@ -1,5 +1,4 @@
 <?xml version="1.0"?>
-<!-- TODO CHECK INERTIAL COLLISION AND FIXED JOINTS" -->
-<robot name="gara" xmlns:xacro="http://ros.org/wiki/xacro">
+<robot name="gara" xmlns:xacro="http://www.ros.org/wiki/xacro">
 	<xacro:include filename="$(find gara_simulation)/urdf/macros.xacro" />
 	<xacro:include filename="$(find gara_simulation)/urdf/gara.gazebo" />
@@ -241,5 +240,4 @@
  	<!-- IMU Joint 	-->
 	<joint name="imu_joint" type="fixed">
-		<axis xyz="0 1 0" />
 		<origin xyz="-0.2 0 ${wheelRadius}" rpy="0 0 0"/>
 		<parent link="chassis"/>

Commit message: Correct an error in the inertial definition in the simulation robot

File: gara_simulation/urdf/gara.xacro (robot description, xacro)
@@ -126,5 +126,5 @@
 	<link name='mast'>
 		<visual name='mast_visual'>
-			<origin xyz="0.0 0 -0.559" rpy="0 0 0"/>
+			<origin xyz="0.0 0 0.55" rpy="0 0 0"/>
 			<geometry>
 				<cylinder radius="0.02" length="1.1"/>
@@ -132,5 +132,5 @@
 		</visual>
 		<collision name='collision'>
-			<origin xyz="0.0 0 -0.559" rpy="0 0 0"/>
+			<origin xyz="0.0 0 0.55" rpy="0 0 0"/>
 			<geometry>
 				<cylinder radius="0.02" length="1.1"/>
@@ -138,6 +138,6 @@
 		</collision>
 		<inertial>
-			<origin xyz="0 0 1.1" rpy="0 0 0"/>
-			<mass value="2"/>
+			<origin xyz="0.0 0 0.55" rpy="0 0 0"/>
+			<mass value="0.1"/>
 			<cylinder_inertia
 				m="0.1"
@@ -148,5 +148,5 @@
 	<!-- Mast Joint -->
 	<joint name="mast_hinge" type="fixed" >
-		<origin xyz="0 0 ${wheelRadius+1.1}" rpy="0 0 0"/>
+		<origin xyz="0 0 ${wheelRadius+0.009}" rpy="0 0 0"/>
 		<parent link="chassis"/>
 		<child link="mast"/>

File: gara_simulation/urdf/macros.xacro (robot description, xacro)
@@ -3,10 +3,10 @@
   <xacro:macro name="cylinder_inertia" params="m r h">
     <inertia
-          ixx="${m*(3*r*r+h*h)/12}"
+          ixx="${(m/12)*(3*r*r+h*h)}"
     			ixy = "0"
     			ixz = "0"
-    			iyy="${m*(3*r*r+h*h)/12}"
+    			iyy="${(m/12)*(3*r*r+h*h)}"
     			iyz = "0"
-    			izz="${m*r*r/2}"/>
+    			izz="${(m/2)*(r*r)}"/>
   </xacro:macro>
   <xacro:macro name="box_inertia" params="m x y z">
