Commit message: Adjust a the mass an intertial parameters

File: gara_simulation/urdf/gara.xacro (robot description, xacro)
@@ -49,4 +49,5 @@
 		</collision>
 		<inertial>
+			<origin xyz="0.0 0 ${casterMass/2.0}" rpy="0 0 0"/>
  			<mass value="${casterMass}"/>
 			<sphere_inertia
@@ -139,7 +140,7 @@
 		<inertial>
 			<origin xyz="0.0 0 0.55" rpy="0 0 0"/>
-			<mass value="0.1"/>
-			<cylinder_inertia
-				m="0.1"
+			<mass value="${mastMass}"/>
+			<cylinder_inertia
+				m="${mastMass}"
 				r="0.02"
 				h="1.1"/>
@@ -166,7 +167,7 @@
 		</collision>
 		<inertial>
-			<mass value="0.1" />
+			<mass value="0.05" />
 			<box_inertia
-				m="0.1"
+				m="0.05"
 				x="0.025"
 				y="0.085"
@@ -180,7 +181,7 @@
 		<child link="camera_link"/>
 	</joint>
-	<!-- Camera RGBD Link 	-->
+	<!-- Camera RGBD Link -->
 	<link name='camera_rgbd_frame'></link>
-	<!-- Camera RGBD Joint -->
+	Camera RGBD Joint
 	<joint name="camera_rgbd_joint" type="fixed" >
 		<origin xyz="0 0 0" rpy="-1.5707963267948966 0 -1.5707963267948966"/>
@@ -188,5 +189,5 @@
     	<child link="camera_rgbd_frame"/>
   	</joint>
-	<!-- Hokuyo Laser Link 	-->
+	<!-- Hokuyo Laser Link -->
 	<link name="hokuyo_link">
   		<visual>
@@ -202,7 +203,7 @@
   		</collision>
   		<inertial>
-		  	<mass value="0.1" />
+		  	<mass value="0.05" />
 			<box_inertia
-				m="0.1"
+				m="0.05"
 				x="0.1"
 				y="0.1"
@@ -230,7 +231,7 @@
 		</collision>
 		<inertial>
-		  	<mass value="0.1" />
+		  	<mass value="0.05" />
 			<box_inertia
-				m="0.1"
+				m="0.05"
 				x="0.01"
 				y="0.01"
@@ -238,5 +239,5 @@
 		</inertial>
 	</link>
- 	<!-- IMU Joint 	-->
+ 	<!-- IMU Joint -->
 	<joint name="imu_joint" type="fixed">
 		<origin xyz="-0.2 0 ${wheelRadius}" rpy="0 0 0"/>

File: gara_simulation/urdf/gara_dimensions.xacro (robot description, xacro)
@@ -6,13 +6,15 @@
 	<xacro:property name="chassisWidth" value="0.018"/>
 	<xacro:property name="chassisRadius" value="0.25"/>
-	<xacro:property name="chassisMass" value="10"/>
+	<xacro:property name="chassisMass" value="0.5"/>
 	<!-- Robot Caster wheel properties -->
-	<xacro:property name="casterRadius" value="0.0585"/>
-	<xacro:property name="casterMass" value="1"/>
+	<xacro:property name="casterRadius" value="0.058"/>
+	<xacro:property name="casterMass" value="0.1"/>
 	<xacro:property name="casterOffsetX" value="0.091"/>
 	<!-- Differential-drive wheels properties -->
 	<xacro:property name="wheelWidth" value="0.05"/>
 	<xacro:property name="wheelRadius" value="0.125"/>
-	<xacro:property name="wheelMass" value="2"/>
+	<xacro:property name="wheelMass" value="0.1"/>
 	<xacro:property name="wheelOffsetY" value="0.037"/>
+	<!-- Differential-drive wheels properties -->
+	<xacro:property name="mastMass" value="0.1"/>
 </robot>

Commit message: correct hokuyo position

File: gara_simulation/urdf/gara.xacro (robot description, xacro)
@@ -214,5 +214,5 @@
 	<joint name="hokuyo_joint" type="fixed">
     	<axis xyz="0 1 0" />
-  		<origin xyz="0 0 1.1" rpy="0 0 0"/>
+  		<origin xyz="0 0 ${wheelRadius+0.009+1.1}" rpy="0 0 0"/>
   		<parent link="chassis"/>
   		<child link="hokuyo_link"/>

Commit message: Navigation fix the local costmap error

File: gara_simulation/urdf/gara.xacro (robot description, xacro)
@@ -214,5 +214,5 @@
 	<joint name="hokuyo_joint" type="fixed">
     	<axis xyz="0 1 0" />
-  		<origin xyz="0 0 ${wheelRadius+0.009+1.1}" rpy="0 0 0"/>
+  		<origin xyz="0 0 0.3" rpy="0 0 0"/>
   		<parent link="chassis"/>
   		<child link="hokuyo_link"/>
